File: hw/LEDDimmer/pcb/VANDIMMER-8CH-2big.kicad_pcb (KiCad board)
At the start: 2 copper layers, 96.7 x 132.1 mm, 42 parts, among them J1 PWR_IN, J10 BTN1, J11 BTN2, J2 CH1, J3 CH2, J4 CH3, J5 CH4, J6 CH5, J7 CH6, J8 CH7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

Commit message: updates to pcb
Parts:
- moved J11 40.8 mm to (45.7, 88.9), turned to 90 degrees
- moved J10 36.0 mm to (45.7, 83.8), turned to 90 degrees
- moved R18 35.9 mm to (40.6, 88.9), turned to 180 degrees
- moved R17 32.3 mm to (40.6, 83.8), turned to 180 degrees
- moved U2 31.9 mm to (47.5, 54.1), turned to 90 degrees
- moved C2 27.0 mm to (48.3, 96.5)
- moved U1 27.0 mm to (53.3, 107.6)
- moved C1 27.0 mm to (48.3, 101.6)
- moved J1 13.9 mm to (50.8, 152.4), turned to 0 degrees
- moved C4 13.4 mm to (49.8, 137.2)
Routing:
- net GND: track 551.4 -> 421.2 mm, vias 2 -> 0
- net CH8: track 61.1 -> 96.3 mm
- net +3.3V: track 109.5 -> 143.9 mm
- net CH7: track 48.7 -> 80.0 mm
- net CH6: track 36.0 -> 63.4 mm
- net Net-(J11-Pin_1): track 58.8 -> 81.3 mm
- net CH5: track 24.1 -> 46.2 mm
- net CH4: track 14.3 -> 34.4 mm
- net Net-(J10-Pin_1): track 62.6 -> 72.3 mm
- net VIN: track 320.7 -> 312.6 mm
- net CH3: track 18.3 -> 24.3 mm
- net CH2: track 29.2 -> 32.0 mm
- net CH1: track 42.6 -> 41.1 mm, vias 0 -> 2
Other:
- board size 96.7 x 132.1 mm -> 106.7 x 132.1 mm
