File: hw/VDDimmer/Power.kicad_sch (KiCad schematic)
At the start: 33 parts, among them J2 VIN 12V, Q5 SUD50P06-15, U2 AP63301WU-7, U3 BL1117-33CX

Commit message: Re-source F1: JLC will not assemble the LUTE fuse
JLC's parts matcher accepted 34 of 35 BOM lines and left F1 unselected. The part
is real -- LUTE LTC2410-1800TSK (C54824501) is a genuine 2410 surface-mount fuse,
8 A, 250 V, 22k in stock -- but it carries no EasyEDA library data
(has_easyeda_footprint false, datasheet null, lcsc_url null). It is a catalogue
part, not an assembly part.

Replaced with BHFUSE BSMD2410C-1800T (C49305064), which has EasyEDA data and is
better on every axis that matters:

                    LUTE C54824501      BHFUSE C49305064
  rating            8 A                 8 A
  voltage (DC)      250 V               250 V
  interrupt         50 A                100 A@350VAC
  melting I2t       115.2               192
  price             $0.0946             $0.0684
  stock             22081               8740
  EasyEDA data      no                  yes

Deliberately still 8 A. The 2026-08-29 decision picked 8 A because it opens BELOW
the 7.5 A blade fuse the spec requires upstream; a 10 A part (C49328463, same
BHFUSE family, 41k stock) would open after it and leave F1 useless as the
board-level backup. The 5 A parts are the opposite problem -- 3.75 A usable after
25% derating, under the 5 A board cap, so they would nuisance-blow.

Higher I2t (192 vs 115.2) makes it slightly slower, which is the right direction
behind a blade fuse and on a board with 10 uF-class input capacitance.

Body is 6.1 x 2.6 mm against the LUTE's 6.1 x 2.5. The land's pads are
1.80 x 2.90 mm each, so it drops in.

Also noted while investigating: D7 (WS2812B) and U1 (ESP32-S3 module) show as
"Standard only" in JLC's matcher. That is not an error -- Economic PCBA places
only a restricted parts list, and a module plus an addressable LED both require
Standard. Standard must be selected for this board regardless.

ERC 0. Bundle rebuilt: 100.00 x 84.00 mm, 247 drills, 78/78 designators, every
line carrying an LCSC code.

Co-Authored-By: Claude Opus 5 (1M context) <noreply@anthr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
Parts:
- F1: Assembly 8 A fuse - sized for the 5 A board cap with 25% continuous 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 -> 8 A fuse, 250 V, 100 A interrupt, I2t 192. Replaces LUTE LT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; LCSC C54824501 -> C49305064; MPN LTC2410-1800TSK -> BSMD2410C-1800T; Manufacturer LUTE -> BHFUSE
Changed lines of the file:
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@@
 			)
 		)
-		(property "Assembly" "8 A fuse - sized for the 5 A board cap with 25% continuous derating; opens below the 7.5 A blade fuse upstream"
+		(property "Assembly" "8 A fuse, 250 V, 100 A interrupt, I2t 192. Replaces LUTE LTC2410-1800TSK (C54824501) which JLC would not select for assembly - that part has no EasyEDA library data (has_easyeda_footprint false), so it is catalogue-only. Keep 8 A: it must open BELOW the 7.5 A blade fuse the spec requires upstream, so 10 A is not a substitute"
 			(at 59.69 44.45 0)
 			(hide yes)
@@
 			)
 		)
-		(property "LCSC" "C54824501"
+		(property "LCSC" "C49305064"
 			(at 59.69 44.45 0)
 			(hide yes)
@@
 			)
 		)
-		(property "MPN" "LTC2410-1800TSK"
+		(property "MPN" "BSMD2410C-1800T"
 			(at 59.69 44.45 0)
 			(hide yes)
@@
 			)
 		)
-		(property "Manufacturer" "LUTE"
+		(property "Manufacturer" "BHFUSE"
 			(at 59.69 44.45 0)
 			(hide yes)
