File: hw/VDDimmer/MCU.kicad_sch (KiCad schematic)
At the start: 24 parts, among them J1 USB-C 16P, J11 BTN1, J12 BTN2, J13 EXP 3V3/GND/SDA/SCL/EN/IO0, J14 UART1 3V3/GND/TX/RX, U1 ESP32-S3-WROOM-1-N16R8

Commit message: Rev B outline, mounting holes and antenna keepout
Mounting holes H1-H4 go M3 -> M2.5 per spec section 5.1. The plan does not
spell this out, but the M2.5 decision is meaningless while the footprints are
still MountingHole_3.2mm_M3. The M2.5 footprint measures 2.7 mm NPTH drill
and a 2.95 mm courtyard radius = 5.90 mm keepout diameter, matching the spec
figure exactly. The smaller keepout is the point: it leaves more copper at the
plane necks, where Rev A pinched to 1.9 mm ~ 3.8 A at H2/H3.

H1-H4 are schematic symbols, not PCB-only items, so the footprint change is
made in MCU.kicad_sch and reaches the board via Update PCB from Schematic at
the start of Phase 4. Same route carries U1's -1U -> -1 swap, which Task 2
made in the schematic but which has not yet reached the .kicad_pcb.

Antenna keepout measured, not remembered, per spec section 4: the WROOM-1
footprint carries its own 48.00 x 21.00 mm rule area spanning F.Cu, B.Cu and
In1..In30.Cu, so it already covers the new 4-layer stack. Rotation 270 puts it
at +x; verified in pcbnew across all four rotations rather than derived.

U1 target is (193.50, uy) rot 270: keepout 100% off board, every pad on board
with 1.24 mm to the edge, and 6.30 mm of module body overhanging - the antenna
section, which is Espressif's option (1).

Outline stays 100 x 84 mm. Figures recorded in analysis/rev-b-task8-geometry.md
so Phase 4 applies measured numbers instead of re-deriving them.

ERC re-run after the footprint changes: 0 violations.

Co-Authored-By: Claude Opus 5 (1M context) <noreply@anthropic.com>
Claude-Session: https://claude.ai/code/session_01YZHVU8aymL4RkLeCfwomwj
Parts:
- H1, H2, H3, H4: footprint MountingHole:MountingHole_3.2mm_M3 -> MountingHole:MountingHole_2.7mm_M2.5
Changed lines of the file:
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@@
 			)
 		)
-		(property "Footprint" "MountingHole:MountingHole_3.2mm_M3"
+		(property "Footprint" "MountingHole:MountingHole_2.7mm_M2.5"
 			(at 90.17 250.19 0)
 			(hide yes)
@@
 			)
 		)
-		(property "Footprint" "MountingHole:MountingHole_3.2mm_M3"
+		(property "Footprint" "MountingHole:MountingHole_2.7mm_M2.5"
 			(at 64.77 250.19 0)
 			(hide yes)
@@
 			)
 		)
-		(property "Footprint" "MountingHole:MountingHole_3.2mm_M3"
+		(property "Footprint" "MountingHole:MountingHole_2.7mm_M2.5"
 			(at 39.37 250.19 0)
 			(hide yes)
@@
 			)
 		)
-		(property "Footprint" "MountingHole:MountingHole_3.2mm_M3"
+		(property "Footprint" "MountingHole:MountingHole_2.7mm_M2.5"
 			(at 115.57 250.19 0)
 			(hide yes)
